Commit message: Add files via upload
机械臂现在有轻微振荡，gazebo里机械爪显示不完全（下一步尝试使用pytho脚本控制不要使用rviz）

File: robotiq_2f_85_gripper_visualization/urdf/robotiq_arg2f_85_model_macro.xacro (robot description, xacro)
@@ -151,5 +151,5 @@
       <child link="${prefix}${fingerprefix}_inner_finger" />
       <axis xyz="1 0 0" />
-      <limit lower="0" upper="0.7" velocity="2.0" effort="1000" />
+      <limit lower="0" upper="0.445" velocity="2.0" effort="1000" />
       <mimic joint="${prefix}finger_joint" multiplier="-1" offset="0" />
     </joint>
